Commit message: base_link adjusted

File: urdf/mobile_and_arm.xacro (robot description, xacro)
@@ -236,5 +236,5 @@
   <link name="base_link">
     <visual>
-      <origin xyz="0 0 0" rpy="${M_PI/2} 0 0" /> <!-- rotate PI/2 -->
+      <origin xyz="0 0 0.05" rpy="${M_PI/2} 0 0" /> <!-- rotate PI/2 -->
       <geometry>
 	       <box size="0.1 0.1 0.1" />
