Commit message: [model ultimated] working

File: urdf/mobile_and_arm.urdf (robot description, URDF)
Before this commit: robot mobile_and_arm, 21 links, 20 joints
Links:
- removed link bottom_link
Joints:
- removed joint bottom_joint

File: urdf/mobile_and_arm.xacro (robot description, xacro)
@@ -228,28 +228,4 @@
   <wheel fb="front" lr="left" parent="base1_link" translateX="0" translateY="-0.5" flipY="1"/>
 <!-- ///////////////////////////////////////////////////////////////////////////////////////////////////////////////////// -->
-  <joint name="bottom_joint" type="fixed">
-    <origin xyz="0 0 0" rpy="0 0 0" />
-    <parent link="base_link"/>
-    <child link="bottom_link"/>
-  </joint>
-  <link name="bottom_link">
-    <visual>
-      <origin xyz=" 0 0 -0.04"  rpy="0 0 0"/>
-      <geometry>
-	       <box size="1 1 0.02" />
-      </geometry>
-      <material name="azure" />
-    </visual>
-    <collision>
-      <origin xyz=" 0 0 -0.04"  rpy="0 0 0"/>
-      <geometry>
-	       <box size="1 1 0.02" />
-      </geometry>
-      </collision>>
-  </link>
-  <gazebo reference="bottom_link">
-    <material>Gazebo/White</material>
-  </gazebo>
-<!-- ///////////////////////////////////////////////////////////////////////////////////////////////////////////////////// -->
   <joint name="bases_joint" type="fixed">
     <origin xyz="0 0 0" rpy="0 0 0" />

Commit message: camera sensor put in place

File: urdf/mobile_and_arm.urdf (robot description, URDF)
Before this commit: robot mobile_and_arm, 20 links, 19 joints
Joints:
- joint rgbd_camera_joint: origin xyz=0.15 0.0 0.8 rpy=0 1.3089969389957472 0 -> xyz=0.0 0.075 0.05 rpy=0 0.0 1.5707963267948966

File: urdf/mobile_and_arm.xacro (robot description, xacro)
@@ -550,5 +550,5 @@
   <!-- Define RGB-D sensor -->
   <xacro:xtion_pro_live name="rgbd_camera" parent="base">
-    <origin xyz="0.15 0.0 0.8" rpy="0 ${75.0 * deg_to_rad} 0"/>
+    <origin xyz="0.0 0.075 0.05" rpy="0 ${0 * deg_to_rad} ${90 * deg_to_rad}"/>
     <origin xyz="0 0 0" rpy="${-90.0 * deg_to_rad} 0 ${-90.0 * deg_to_rad}"/>
   </xacro:xtion_pro_live>
